File: Dough/dough/power managment.kicad_sch (KiCad schematic)
At the start: 28 parts, among them J1 BATT IN, J10 USB_ESP32, J3 USB_RP2040, Q3 AO3401A, U3 AZ1084-5.0, U4 TLV1117-33, U5 LM4040DBZ-3

Commit message: pre prod 1
Parts:
- added D8, D9: LED, LED_SMD:LED_0603_1608Metric_Pad1.05x0.95mm_HandSolder, symbol Device:LED
- added R42, R43: 10k, Resistor_SMD:R_0603_1608Metric_Pad0.98x0.95mm_HandSolder, symbol Device:R_Small
Connections:
- net GND: now also D8.1 (K), D9.1 (K)
- net at D4.2 (A), J10.1 (VBUS): now also R43.2
- net at D6.2 (A), J3.1 (VBUS): now also R42.2
- new net: D9.2 (A), R43.1
- new net: D8.2 (A), R42.1
