File: Dough/dough/rp2040 section.kicad_sch (KiCad schematic)
At the start: 70 parts, among them J11 Conn_01x10_Pin, J2 Conn_01x05_Pin, J4 servo 6, J5 servo 1, J6 servo 2, J7 servo 3, J8 servo 4, J9 servo 5, Q2 2N7002, Q5 2N7002, SW1 2040 RST, SW301 2040 BOOTSEL, U1 W25Q32JVSS, U11 25SH-B-04-TS, U2 RP2040, U6 BMP581, U7 MMC5633NJL, U8 BMI160, Y1 Crystal

Commit message: started routing
Parts:
- removed C21: 100n, Capacitor_SMD:C_0603_1608Metric_Pad1.08x0.95mm_HandSolder, symbol Device:C_Small
Changed lines of the file:
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@@
 	)
 	(junction
-		(at 252.095 81.915)
-		(diameter 0)
-		(color 0 0 0 0)
-	)
-	(junction
 		(at 194.945 39.37)
 		(diameter 0)
@@
 	)
 	(junction
-		(at 263.525 78.74)
-		(diameter 0)
-		(color 0 0 0 0)
-	)
-	(junction
 		(at 205.74 128.27)
 		(diameter 0)
@@
 	(wire
 		(pts
-			(xy 252.095 81.915) (xy 256.54 81.915)
-		)
-		(stroke
-			(width 0)
-			(type default)
-		)
-	)
-	(wire
-		(pts
 			(xy 239.395 15.24) (xy 239.395 17.145)
 		)
@@
 	(wire
 		(pts
-			(xy 263.525 81.915) (xy 263.525 78.74)
-		)
-		(stroke
-			(width 0)
-			(type default)
-		)
-	)
-	(wire
-		(pts
 			(xy 198.755 98.425) (xy 197.485 98.425)
 		)
@@
 	(wire
 		(pts
-			(xy 263.525 78.74) (xy 264.795 78.74)
-		)
-		(stroke
-			(width 0)
-			(type default)
-		)
-	)
-	(wire
-		(pts
 			(xy 43.18 143.51) (xy 38.1 143.51)
 		)
@@
 	(wire
 		(pts
-			(xy 252.095 81.915) (xy 252.095 82.55)
+			(xy 252.095 80.645) (xy 252.095 82.55)
 		)
 		(stroke
@@
 	(wire
 		(pts
-			(xy 252.095 80.645) (xy 252.095 81.915)
-		)
-		(stroke
-			(width 0)
-			(type default)
-		)
-	)
-	(wire
-		(pts
 			(xy 88.265 81.915) (xy 113.03 81.915)
 		)
@@
 	(wire
 		(pts
-			(xy 261.62 78.74) (xy 263.525 78.74)
+			(xy 261.62 78.74) (xy 264.795 78.74)
 		)
 		(stroke
@@
 	(wire
 		(pts
-			(xy 261.62 81.915) (xy 263.525 81.915)
-		)
-		(stroke
-			(width 0)
-			(type default)
-		)
-	)
-	(wire
-		(pts
 			(xy 119.38 46.99) (xy 125.095 46.99)
 		)
@@
 					(unit 1)
 				)
-			)
-		)
-	)
-	(symbol
-		(lib_id "Device:C_Small")
-		(at 259.08 81.915 270)
-		(unit 1)
-		(exclude_from_sim no)
-		(in_bom yes)
-		(on_board yes)
-		(dnp no)
-		(property "Reference" "C21"
-			(at 259.08 84.455 90)
-			(effects
-				(font
-					(size 1.27 1.27)
-				)
-			)
-		)
-		(property "Value" "100n"
-			(at 259.08 86.36 90)
-			(effects
-				(font
-					(size 1.27 1.27)
-				)
-			)
-		)
-		(property "Footprint" "Capacitor_SMD:C_0603_1608Metric_Pad1.08x0.95mm_HandSolder"
-			(at 259.08 81.915 0)
-			(effects
-				(font
-					(size 1.27 1.27)
-				)
-				(hide yes)
-			)
-		)
-		(property "Datasheet" "~"
-			(at 259.08 81.915 0)
-			(effects
-				(font
-					(size 1.27 1.27)
-				)
-				(hide yes)
-			)
-		)
-		(property "Description" "Unpolarized capacitor, small symbol"
-			(at 259.08 81.915 0)
-			(effects
-				(font
-					(size 1.27 1.27)
-				)
-				(hide yes)
-			)
-		)
-		(pin "2"
-		)
-		(pin "1"
-		)
-		(instances
-			(project "dough"
-				(path "/4fefffc5-b577-4f4a-9ede-53ada2aa57cf/ead411db-855b-49b3-973c-12a7f8331e1f"
-					(reference "C21")
-					(unit 1)
-				)

Commit message: pre prod 1
Parts:
- removed C29: 100n, Capacitor_SMD:C_0603_1608Metric_Pad1.08x0.95mm_HandSolder, symbol Device:C_Small
- added JP3: ~, Jumper:SolderJumper-3_P1.3mm_Open_RoundedPad1.0x1.5mm, symbol Jumper:SolderJumper_3_Open
- added R44: 10k, Resistor_SMD:R_0603_1608Metric_Pad0.98x0.95mm_HandSolder, symbol Device:R_Small
Connections:
- net +3V3: now also R44.1
- net GND: now also J4.1 (Pin_1), J5.1 (Pin_1), J6.1 (Pin_1), J7.1 (Pin_1), J8.1 (Pin_1), J9.1 (Pin_1), JP3.1 (A); no longer C11.2, SW1.1, SW301.1
- net LED_B: now also U2.36 (GPIO24)
- net LED_G: now also U2.35 (GPIO23)
- net LED_R: now also U2.34 (GPIO22)
- new net: JP3.3 (B), R44.2
- new net BUTTONS: C11.2, JP3.2 (C), SW1.1, SW301.1
Other:
- moved on the sheet: R13
