File: Dough/dough/dough.kicad_pcb (KiCad board)
At the start: 4 copper layers, 50 x 70 mm, 130 parts, among them J1 BATT IN, J10 USB_ESP32, J11 Conn_01x10_Pin, J12 Conn_01x10_Pin, J2 Conn_01x05_Pin, J3 USB_RP2040, J4 servo 6, J401 SD CARD, J5 servo 1, J6 servo 2, J7 servo 3, J8 servo 4, J9 servo 5, Q1 2N7002, Q2 2N7002, Q3 AO3401A, Q4 2N7002, SW1 2040 RST, SW2 ESP32 BOOT, SW301 2040 BOOTSEL, SW4 ESP32 RST, U1 W25Q32JVSS, U11 25SH-B-04-TS, U2 RP2040, U3 AZ1084-5.0, U4 TLV1117-33, U5 LM4040DBZ-3, U6 BMP581, U7 MMC5633NJL, U8 BMI160, U9 ESP32-S3-WROOM-1, Y1 Crystal

Commit message: started routing
Parts:
- removed C12, C15, C17, C21, C34, C35: 100n, Capacitor_SMD:C_0603_1608Metric_Pad1.08x0.95mm_HandSolder
- added Q5: 2N7002, Package_TO_SOT_SMD:SOT-23, B.Cu at (131.8, 61.4)
- added R40: 27, Resistor_SMD:R_0603_1608Metric_Pad0.98x0.95mm_HandSolder, B.Cu at (113.8, 57.6)
- added R41: 27, Resistor_SMD:R_0603_1608Metric_Pad0.98x0.95mm_HandSolder, B.Cu at (115.3, 57.6)
- C11, C18, C25, C401, C402, C405, R14, R15, R16, R28, R29, R30, R31, R32: moved to F.Cu
- JP2, Q1, Q4: moved to B.Cu
- R12: value 4.7k -> 1k
- R13: value 4.7k -> 10k
- moved D6 150.7 mm to (105.5, 64.7)
- moved U5 149.0 mm to (116.0, 73.2)
- moved D3 138.9 mm to (116.3, 88.2)
- moved C3 137.3 mm to (113.8, 95.7), turned to -90 degrees
- moved C2 137.1 mm to (113.8, 91.2), turned to 90 degrees
- moved C1 135.9 mm to (115.3, 91.2), turned to 90 degrees
- moved C13 135.6 mm to (114.8, 78.2), turned to 90 degrees
- moved C4 135.6 mm to (115.3, 95.7), turned to -90 degrees
- moved Q2 133.1 mm to (128.6, 55.9)
- moved C14 129.9 mm to (116.0, 69.9), turned to -90 degrees
- moved R37 129.4 mm to (112.3, 89.4), turned to 90 degrees
- moved R2 129.2 mm to (116.8, 79.7), turned to 90 degrees
- moved R1 129.1 mm to (116.8, 83.2), turned to 90 degrees
- moved R5 128.3 mm to (113.3, 73.2), turned to 90 degrees
- moved D2 127.1 mm to (109.8, 92.7), turned to 0 degrees
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Connections:
- C11 pad 1: GND -> Net-(Q5-S)
- C11 pad 2: +3V3 -> GND
- R11 pad 2: Net-(U2-RUN) -> Net-(Q5-S)
- R12 pad 1: +3V3 -> RP2040_RST
- R12 pad 2: SDA1 -> Net-(Q5-G)
- R13 pad 1: +3V3 -> GND
- R13 pad 2: SCL1 -> Net-(Q5-G)
- R38 pad 1: ESP32_RST -> ESP32_BOOT
- SW1 pad 2: Net-(U2-RUN) -> Net-(Q5-S)
- U2 pad 26: Net-(U2-RUN) -> Net-(Q5-S)
- U2 pad 30: unconnected-(U2-GPIO19-Pad30) -> ESP32_BOOT
- U9 pad 13: USB2_D- -> Net-(U9-IO19)
- U9 pad 14: USB2_D+ -> Net-(U9-IO20)
- U9 pad 8: unconnected-(U9-IO15-Pad8) -> RP2040_RST
Routing:
- net GND: track 0.00 -> 232.6 mm, vias 0 -> 2
- net +3V3: track 0.00 -> 135.8 mm, vias 0 -> 8
- net +5V: track 0.00 -> 64.3 mm
- net Net-(JP2-C): track 0.00 -> 60.7 mm
- net SER_6: track 0.00 -> 41.9 mm, vias 0 -> 1
- net SER_1: track 0.00 -> 40.7 mm, vias 0 -> 1
- net SER_5: track 0.00 -> 40.2 mm, vias 0 -> 1
- net SER_4: track 0.00 -> 39.5 mm, vias 0 -> 1
- net Net-(U2-XIN): track 0.00 -> 37.0 mm, vias 0 -> 2
- net SER_3: track 0.00 -> 32.8 mm, vias 0 -> 1
- net SER_2: track 0.00 -> 32.4 mm, vias 0 -> 1
- net Net-(U2-XOUT): track 0.00 -> 31.3 mm, vias 0 -> 2
- net +BATT: track 0.00 -> 28.1 mm
- net USB1_D+: track 0.00 -> 28.0 mm, vias 0 -> 2
- net SD_CD: track 0.00 -> 26.3 mm, vias 0 -> 2
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Other:
- board size 50 x 70 mm -> 50 x 72.5 mm

Commit message: pre prod 1
Parts:
- removed C29: 100n, Capacitor_SMD:C_0603_1608Metric_Pad1.08x0.95mm_HandSolder
- added D8: LED, LED_SMD:LED_0603_1608Metric_Pad1.05x0.95mm_HandSolder, F.Cu at (105.9, 67.8)
- added D9: LED, LED_SMD:LED_0603_1608Metric_Pad1.05x0.95mm_HandSolder, F.Cu at (139.6, 67.8)
- added JP3: ~, Jumper:SolderJumper-3_P1.3mm_Open_RoundedPad1.0x1.5mm, B.Cu at (106.1, 73.1)
- added R35: 10k, Resistor_SMD:R_0603_1608Metric_Pad0.98x0.95mm_HandSolder, B.Cu at (107.8, 43.1)
- added R39: 10k, Resistor_SMD:R_0603_1608Metric_Pad0.98x0.95mm_HandSolder, B.Cu at (137.6, 57.1)
- added R42: 10k, Resistor_SMD:R_0603_1608Metric_Pad0.98x0.95mm_HandSolder, B.Cu at (105.7, 66.6)
- added R43: 10k, Resistor_SMD:R_0603_1608Metric_Pad0.98x0.95mm_HandSolder, B.Cu at (139.5, 66.4)
- added R44: 10k, Resistor_SMD:R_0603_1608Metric_Pad0.98x0.95mm_HandSolder, B.Cu at (110.5, 74.6)
- moved TP2 24.3 mm to (123.0, 65.2)
- moved TP1 22.4 mm to (125.6, 60.0)
- moved TP4 10.4 mm to (134.8, 65.3)
- moved TP3 8.02 mm to (134.8, 67.8)
- moved R11 3.75 mm to (120.0, 83.7)
- moved D7 3.51 mm to (134.4, 56.1)
- moved TP6 2.70 mm to (136.7, 71.0)
- moved TP5 2.52 mm to (134.2, 71.0)
- moved C31 0.80 mm to (125.3, 73.9)
- moved C10 0.72 mm to (114.3, 69.2)
- moved C14 0.72 mm to (115.8, 69.2)
- moved R19 0.17 mm to (123.0, 82.3)
- moved R26 0.07 mm to (130.8, 65.3)
Connections:
- C11 pad 2: GND -> BUTTONS
- C25 pad 2: GND -> BUTTONS
- C402 pad 2: GND -> BUTTONS
- J4 pad 1: Net-(J4-Pin_1) -> GND
- J5 pad 1: Net-(J4-Pin_1) -> GND
- J6 pad 1: Net-(J4-Pin_1) -> GND
- J7 pad 1: Net-(J4-Pin_1) -> GND
- J8 pad 1: Net-(J4-Pin_1) -> GND
- J9 pad 1: Net-(J4-Pin_1) -> GND
- SW1 pad 1: GND -> BUTTONS
- SW2 pad 1: GND -> BUTTONS
- SW301 pad 1: GND -> BUTTONS
- SW4 pad 1: GND -> BUTTONS
- U2 pad 34: unconnected-(U2-GPIO22-Pad34) -> LED_R
- U2 pad 35: unconnected-(U2-GPIO23-Pad35) -> LED_G
- U2 pad 36: unconnected-(U2-GPIO24-Pad36) -> LED_B
- U9 pad 10: unconnected-(U9-IO17-Pad10) -> SDA1
- U9 pad 11: unconnected-(U9-IO18-Pad11) -> SCL1
- U9 pad 15: unconnected-(U9-IO3-Pad15) -> SER_3
- U9 pad 38: unconnected-(U9-IO2-Pad38) -> SER_2
- U9 pad 39: unconnected-(U9-IO1-Pad39) -> SER_1
- U9 pad 9: unconnected-(U9-IO16-Pad9) -> SER_4
Routing:
- net GND: track 232.6 -> 493.1 mm, vias 2 -> 12
- net +3V3: track 135.8 -> 269.0 mm, vias 8 -> 11
- net +5V: track 64.3 -> 153.9 mm, vias 0 -> 4
- net BUTTONS: track 0.00 -> 82.2 mm, vias 0 -> 2
- net SCL0: track 3.61 -> 77.8 mm, vias 1 -> 4
- net ADC2: track 0.00 -> 72.2 mm, vias 0 -> 3
- net USB2_D+: track 0.00 -> 70.8 mm, vias 0 -> 3
- net USB2_D-: track 0.00 -> 67.6 mm, vias 0 -> 3
- net ADC0: track 0.00 -> 66.9 mm, vias 0 -> 4
- net SDA0: track 3.20 -> 69.9 mm, vias 1 -> 3
- net ADC1: track 0.00 -> 66.0 mm, vias 0 -> 4
- net GPIO4_esp: track 0.00 -> 62.2 mm, vias 0 -> 1
- net SPI0_CS2: track 0.00 -> 60.7 mm, vias 0 -> 3
- net GPIO5_esp: track 0.00 -> 59.2 mm, vias 0 -> 1
- net GPIO6_esp: track 0.00 -> 57.1 mm, vias 0 -> 1
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- added copper zone on B.Cu, net GND
- added copper zone on F.Cu, net GND
Other:
- board text added: "Dough"
- board text added: "V 1.0"

Commit message: V1.0 pre prod
Parts:
- removed Y1: Crystal, Crystal:Crystal_SMD_FOX_FE-2Pin_7.5x5.0mm_HandSoldering
- added C12: 100n, Capacitor_SMD:C_0603_1608Metric_Pad1.08x0.95mm_HandSolder, B.Cu at (130.5, 80.6)
- added D10: D_Schottky, Diode_SMD:D_SOD-323_HandSoldering, F.Cu at (110.1, 95.8)
- added J13: 5v, 25SH_B_02_TS:CONN2_H-B-02-TS_ADM, F.Cu at (105.3, 97.0)
- added R45: 1k, Resistor_SMD:R_0603_1608Metric_Pad0.98x0.95mm_HandSolder, B.Cu at (128.5, 78.9)
- added R46: 10k, Resistor_SMD:R_0603_1608Metric_Pad0.98x0.95mm_HandSolder, F.Cu at (120.8, 94.0)
- added R47: SDNT1608, Resistor_SMD:R_0603_1608Metric_Pad0.98x0.95mm_HandSolder, F.Cu at (124.2, 94.0)
- added R48: 10k, Resistor_SMD:R_0603_1608Metric_Pad0.98x0.95mm_HandSolder, F.Cu at (110.1, 92.1)
- added X1: ECS-2520MV-xxx-xx, Oscillator:Oscillator_SMD_ECS_2520MV-xxx-xx-4Pin_2.5x2.0mm, B.Cu at (127.1, 68.2)
- C6: value 30p -> 1u
- C7: value 30p -> 100n; moved to F.Cu
- moved C6 21.3 mm to (124.4, 69.9), turned to 45 degrees
- moved C7 20.6 mm to (124.2, 95.7)
- moved R10 15.2 mm to (123.7, 75.8), turned to -45 degrees
- moved J1 3.49 mm to (111.5, 87.0)
- moved TP1 2.62 mm to (123.9, 62.0)
- moved D2 1.10 mm to (108.7, 92.7)
- moved C31 0.42 mm to (125.0, 74.2)
Connections:
- C6 pad 1: Net-(C6-Pad1) -> GND
- C6 pad 2: Net-(U2-XIN) -> +3V3
- C7 pad 1: Net-(C7-Pad1) -> ADC2
- C7 pad 2: Net-(U2-XOUT) -> GND
- J11 pad 4: ADC2 -> unconnected-(J11-Pin_4-Pad4)
- J2 pad 1: +5V -> GND
- J2 pad 5: GND -> +5V
- R10 pad 1: Net-(C6-Pad1) -> +3V3
- R10 pad 2: Net-(C7-Pad1) -> Net-(X1-Tri-State)
- U2 pad 21: Net-(U2-XOUT) -> unconnected-(U2-XOUT-Pad21)
- U8 pad 12: +3V3 -> Net-(U8-CSB)
Routing:
- net Net-(U2-XOUT): track 41.9 -> 0.00 mm, vias 2 -> 0
- net Net-(U2-XIN): track 41.6 -> 6.59 mm, vias 2 -> 1
- net ADC2: track 72.2 -> 42.2 mm, vias 3 -> 2
- net GND: track 493.1 -> 467.4 mm, vias 12 -> 11
- net +5V: track 153.9 -> 165.0 mm, vias 4 -> 6
- net Net-(X1-Tri-State): track 0.00 -> 9.37 mm
- net Net-(C6-Pad1): track 8.53 -> 0.00 mm
- net Net-(C7-Pad1): track 8.15 -> 0.00 mm
- net Net-(U8-CSB): track 0.00 -> 6.61 mm, vias 0 -> 1
- net +3V3: track 269.0 -> 275.4 mm
- net Net-(J13-Pad2): track 0.00 -> 6.33 mm
- net GPIO17: track 51.6 -> 54.0 mm
- net GPIO16: track 48.7 -> 51.0 mm
- net Net-(D2-K): track 11.6 -> 9.49 mm
- net Net-(Q5-S): track 46.6 -> 44.7 mm
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Other:
- board text added: "3V"
- board text added: "5V"
- board text added: "ADC"
- board text added: "BATT"
- board text added: "BOOT"
- board text added: "BUTT"
- board text added: "DIS"
- board text added: "EN"
- board text added: "ESP"
- board text added: "GND"
- board text added: "RP2040"
- board text added: "RST"
- board text added: "S1"
- board text added: "S2"
- board text added: "S3"
- board text added: "S4"
- board text added: "S5"
- board text added: "S6"
- board text added: "batt"

Commit message: dough First production run
Parts:
- added C15: 100n, Capacitor_SMD:C_0603_1608Metric_Pad1.08x0.95mm_HandSolder, B.Cu at (113.5, 81.6)
- added U12: ATA6561-GAQW-N, ATA6561_GAQW:SOIC8_4P9X3P9MC_MCH, B.Cu at (108.9, 81.6)
- moved C402 2.25 mm to (133.9, 62.1)
- moved R44 1.90 mm to (110.5, 76.5)
- moved R42 1.20 mm to (105.6, 67.8)
- moved C18 0.77 mm to (115.6, 75.2)
- moved C31 0.58 mm to (124.7, 74.7)
- moved C19 0.51 mm to (129.3, 69.3), turned to -90 degrees
- moved C8 0.35 mm to (116.6, 76.0)
- moved C6 0.30 mm to (124.4, 70.2)
- moved R21 0.22 mm to (119.0, 75.5)
- moved C403 0.20 mm to (114.0, 49.4)
- moved X1 0.10 mm to (127.2, 68.2)
- moved U5 0.07 mm to (116.1, 73.1)
Connections:
- J12 pad 10: GPIO4_esp -> CANL
- J12 pad 9: GPIO5_esp -> CANH
- U2 pad 11: SER_3 -> SER_1
- U2 pad 8: SER_1 -> SER_3
Routing:
- net +5V: track 165.0 -> 186.4 mm, vias 6 -> 7
- net GPIO5_esp: track 59.2 -> 40.2 mm, vias 1 -> 2
- net CANL: track 0.00 -> 17.7 mm
- net CANH: track 0.00 -> 16.2 mm
- net GPIO4_esp: track 62.2 -> 47.9 mm, vias 1 -> 2
- net BUTTONS: track 82.2 -> 72.9 mm, vias 2 -> 1
- net GND: track 467.4 -> 476.6 mm
- net +3V3: track 275.4 -> 280.2 mm
- net Net-(Q1-S): track 52.4 -> 48.2 mm
- net SCL1: track 57.3 -> 61.3 mm
- net GPIO18: track 51.1 -> 48.3 mm
- net USB1_D-: track 25.7 -> 28.3 mm
- net SPI_BIT3: track 46.3 -> 48.3 mm
- net UART1_RX: track 33.1 -> 31.3 mm
- net USB2_D+: track 70.8 -> 72.4 mm
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Other:
- board text removed: "batt"
